File: audio.sch (KiCad schematic (older format))
At the start: 53 parts, among them J1 ohfilt-10k, J2 chfilt-10k, J3 ohfilten, J4 chfilten, Q11 BC546, Q12 BC546, Q13 BC546, Q14 BC546, U4 TL072

Commit message: assigned footprints
Parts:
- C18, C20, C23, C24, C25, C26: footprint (none) -> Capacitor_THT:C_Disc_D4.3mm_W1.9mm_P5.00mm
- C19, C22, C27, C28, C29, C30, C31, C32, C33, C34: footprint (none) -> Capacitor_THT:C_Disc_D3.4mm_W2.1mm_P2.50mm
- C21: footprint (none) -> Capacitor_THT:CP_Radial_D7.5mm_P2.50mm
Changed lines of the file:
@@
 F 0 "C18" V 1823 2025 50  0000 C CNN
 F 1 "22n" V 1914 2025 50  0000 C CNN
-F 2 "" H 2113 1875 50  0001 C CNN
+F 2 "Capacitor_THT:C_Disc_D4.3mm_W1.9mm_P5.00mm" H 2113 1875 50  0001 C CNN
 F 3 "~" H 2075 2025 50  0001 C CNN
 	1    2075 2025
@@
 F 0 "C27" H 3110 1954 50  0000 R CNN
 F 1 "1n5" H 3110 2045 50  0000 R CNN
-F 2 "" H 3263 1850 50  0001 C CNN
+F 2 "Capacitor_THT:C_Disc_D3.4mm_W2.1mm_P2.50mm" H 3263 1850 50  0001 C CNN
 F 3 "~" H 3225 2000 50  0001 C CNN
 	1    3225 2000
@@
 F 0 "C28" H 3560 1954 50  0000 R CNN
 F 1 "1n5" H 3560 2045 50  0000 R CNN
-F 2 "" H 3713 1850 50  0001 C CNN
+F 2 "Capacitor_THT:C_Disc_D3.4mm_W2.1mm_P2.50mm" H 3713 1850 50  0001 C CNN
 F 3 "~" H 3675 2000 50  0001 C CNN
 	1    3675 2000
@@
 F 0 "C30" V 4802 1675 50  0000 C CNN
 F 1 "1n5" V 4711 1675 50  0000 C CNN
-F 2 "" H 4588 1525 50  0001 C CNN
+F 2 "Capacitor_THT:C_Disc_D3.4mm_W2.1mm_P2.50mm" H 4588 1525 50  0001 C CNN
 F 3 "~" H 4550 1675 50  0001 C CNN
 	1    4550 1675
@@
 F 0 "C23" V 5952 2225 50  0000 C CNN
 F 1 "470p" V 5861 2225 50  0000 C CNN
-F 2 "" H 5738 2075 50  0001 C CNN
+F 2 "Capacitor_THT:C_Disc_D4.3mm_W1.9mm_P5.00mm" H 5738 2075 50  0001 C CNN
 F 3 "~" H 5700 2225 50  0001 C CNN
 	1    5700 2225
@@
 F 0 "C24" V 6673 1425 50  0000 C CNN
 F 1 "220p" V 6764 1425 50  0000 C CNN
-F 2 "" H 6963 1275 50  0001 C CNN
+F 2 "Capacitor_THT:C_Disc_D4.3mm_W1.9mm_P5.00mm" H 6963 1275 50  0001 C CNN
 F 3 "~" H 6925 1425 50  0001 C CNN
 	1    6925 1425
@@
 F 0 "C21" V 6520 975 50  0000 C CNN
 F 1 "33u/6.3v" V 6611 975 50  0000 C CNN
-F 2 "" H 6813 825 50  0001 C CNN
+F 2 "Capacitor_THT:CP_Radial_D7.5mm_P2.50mm" H 6813 825 50  0001 C CNN
 F 3 "~" H 6775 975 50  0001 C CNN
 	1    6775 975
@@
 F 0 "C29" V 4127 1675 50  0000 C CNN
 F 1 "1n5" V 4036 1675 50  0000 C CNN
-F 2 "" H 3913 1525 50  0001 C CNN
+F 2 "Capacitor_THT:C_Disc_D3.4mm_W2.1mm_P2.50mm" H 3913 1525 50  0001 C CNN
 F 3 "~" H 3875 1675 50  0001 C CNN
 	1    3875 1675
@@
 F 0 "C20" V 1823 5025 50  0000 C CNN
 F 1 "22n" V 1914 5025 50  0000 C CNN
-F 2 "" H 2113 4875 50  0001 C CNN
+F 2 "Capacitor_THT:C_Disc_D4.3mm_W1.9mm_P5.00mm" H 2113 4875 50  0001 C CNN
 F 3 "~" H 2075 5025 50  0001 C CNN
 	1    2075 5025
@@
 F 0 "C34" H 3110 4954 50  0000 R CNN
 F 1 "1n5" H 3110 5045 50  0000 R CNN
-F 2 "" H 3263 4850 50  0001 C CNN
+F 2 "Capacitor_THT:C_Disc_D3.4mm_W2.1mm_P2.50mm" H 3263 4850 50  0001 C CNN
 F 3 "~" H 3225 5000 50  0001 C CNN
 	1    3225 5000
@@
 F 0 "C33" H 3560 4954 50  0000 R CNN
 F 1 "1n5" H 3560 5045 50  0000 R CNN
-F 2 "" H 3713 4850 50  0001 C CNN
+F 2 "Capacitor_THT:C_Disc_D3.4mm_W2.1mm_P2.50mm" H 3713 4850 50  0001 C CNN
 F 3 "~" H 3675 5000 50  0001 C CNN
 	1    3675 5000
@@
 F 0 "C31" V 4802 4675 50  0000 C CNN
 F 1 "1n" V 4711 4675 50  0000 C CNN
-F 2 "" H 4588 4525 50  0001 C CNN
+F 2 "Capacitor_THT:C_Disc_D3.4mm_W2.1mm_P2.50mm" H 4588 4525 50  0001 C CNN
 F 3 "~" H 4550 4675 50  0001 C CNN
 	1    4550 4675
@@
 F 0 "C26" V 5952 5225 50  0000 C CNN
 F 1 "470p" V 5861 5225 50  0000 C CNN
-F 2 "" H 5738 5075 50  0001 C CNN
+F 2 "Capacitor_THT:C_Disc_D4.3mm_W1.9mm_P5.00mm" H 5738 5075 50  0001 C CNN
 F 3 "~" H 5700 5225 50  0001 C CNN
 	1    5700 5225
@@
 F 0 "C25" V 6673 4425 50  0000 C CNN
 F 1 "220p" V 6764 4425 50  0000 C CNN
-F 2 "" H 6963 4275 50  0001 C CNN
+F 2 "Capacitor_THT:C_Disc_D4.3mm_W1.9mm_P5.00mm" H 6963 4275 50  0001 C CNN
 F 3 "~" H 6925 4425 50  0001 C CNN
 	1    6925 4425
@@
 F 0 "C32" V 4127 4675 50  0000 C CNN
 F 1 "1n" V 4036 4675 50  0000 C CNN
-F 2 "" H 3913 4525 50  0001 C CNN
+F 2 "Capacitor_THT:C_Disc_D3.4mm_W2.1mm_P2.50mm" H 3913 4525 50  0001 C CNN
 F 3 "~" H 3875 4675 50  0001 C CNN
 	1    3875 4675
@@
 F 0 "C22" H 9615 1346 50  0000 L CNN
 F 1 "0.1u" H 9615 1255 50  0000 L CNN
-F 2 "" H 9538 1150 50  0001 C CNN
+F 2 "Capacitor_THT:C_Disc_D3.4mm_W2.1mm_P2.50mm" H 9538 1150 50  0001 C CNN
 F 3 "~" H 9500 1300 50  0001 C CNN
 	1    9500 1300
@@
 F 0 "C19" H 9615 1696 50  0000 L CNN
 F 1 "0.1u" H 9615 1605 50  0000 L CNN
-F 2 "" H 9538 1500 50  0001 C CNN
+F 2 "Capacitor_THT:C_Disc_D3.4mm_W2.1mm_P2.50mm" H 9538 1500 50  0001 C CNN
 F 3 "~" H 9500 1650 50  0001 C CNN
 	1    9500 1650
